File: 68k_breakout_3v3.kicad_sch (KiCad schematic)
At the start: 4 parts, among them J1 Conn_02x32_Odd_Even, J2 Conn_02x02_Odd_Even, U1 68000D_PLUG, U2 68000D

Commit message: Initial layout complete
Parts:
- removed J1: Conn_02x32_Odd_Even, Connector_PinHeader_2.54mm:PinHeader_2x32_P2.54mm_Vertical, symbol Connector_Generic:Conn_02x32_Odd_Even
- added C1, C2, C3, C4, C5, C6, C7, C8: 100n, Capacitor_SMD:C_0805_2012Metric_Pad1.18x1.45mm_HandSolder, symbol Device:C
- added C10, C9: 1u, Capacitor_SMD:C_0805_2012Metric_Pad1.18x1.45mm_HandSolder, symbol Device:C
- added IC1, IC2, IC3, IC4, IC5, IC6, IC7, IC8: SN74CB3T3245DW, Package_SO:TSSOP-20_4.4x6.5mm_P0.65mm, symbol SN74CB3T3245DW:SN74CB3T3245DW
- added J1: Conn_02x02_Odd_Even, Connector_PinSocket_2.54mm:PinSocket_2x02_P2.54mm_Vertical, symbol Connector_Generic:Conn_02x02_Odd_Even
- added J3, J4: Conn_02x20_Odd_Even, Connector_PinHeader_2.54mm:PinHeader_2x20_P2.54mm_Vertical, symbol Connector_Generic:Conn_02x20_Odd_Even
- added RN1, RN2: 10k, Resistor_SMD:R_Array_Convex_4x0603, symbol Device:R_Pack04
- added U3: LM1117-3.3, Package_TO_SOT_SMD:SOT-223-3_TabPin2, symbol Regulator_Linear:LM1117-3.3
Connections:
- net +5V: now also U1.49 (VCC), C9.1, U3.3 (VI)
- net A1: now also IC4.9 (A8)
- net A10: now also IC5.7 (A6)
- net A11: now also IC5.6 (A5)
- net A12: now also IC5.5 (A4)
- net A13: now also IC5.4 (A3)
- net A14: now also IC5.3 (A2)
- net A15: now also IC5.2 (A1)
- net A16: now also IC6.9 (A8)
- net A17: now also IC6.8 (A7)
- net A18: now also IC6.7 (A6)
- net A19: now also IC6.6 (A5)
- net A2: now also IC4.8 (A7)
- net A20: now also IC6.5 (A4)
- net A21: now also IC6.4 (A3)
- net A22: now also IC6.3 (A2)
- net A23: now also IC6.2 (A1)
- net A3: now also IC4.7 (A6)
- net A4: now also IC4.6 (A5)
- net A5: now also IC4.5 (A4)
- net A6: now also IC4.4 (A3)
- net A7: now also IC4.3 (A2)
- net A8: now also IC5.9 (A8)
- net A9: now also IC5.8 (A7)
- net AS: now also IC1.9 (A8)
- net BERR: now also IC3.3 (A2)
- net BG: now also IC1.4 (A3)
- net BGACK: now also IC1.3 (A2)
- net BR: now also IC1.2 (A1)
- net CLK: now also IC3.9 (A8)
- net D0: now also IC7.2 (A1)
- net D1: now also IC7.3 (A2)
- net D10: now also IC8.7 (A6)
- net D11: now also IC8.6 (A5)
- net D12: now also IC8.5 (A4)
- net D13: now also IC8.4 (A3)
- net D14: now also IC8.3 (A2)
- net D15: now also IC8.2 (A1)
- net D2: now also IC7.4 (A3)
- net D3: now also IC7.5 (A4)
- net D4: now also IC7.6 (A5)
- net D5: now also IC7.7 (A6)
- net D6: now also IC7.8 (A7)
- net D7: now also IC7.9 (A8)
- net D8: now also IC8.9 (A8)
- net D9: now also IC8.8 (A7)
- net DTACK: now also IC1.5 (A4)
- net E: now also IC3.5 (A4)
- net FC0: now also IC2.4 (A3)
- net FC1: now also IC2.5 (A4)
- net FC2: now also IC2.6 (A5)
- net GND: now also U1.16 (GND), C1.2, C10.2, C2.2, C3.2, C4.2, C5.2, C6.2, C7.2, C8.2, C9.2, IC1.10 (GND), IC2.10 (GND), IC3.10 (GND), IC4.10 (GND), IC5.10 (GND), IC6.10 (GND), IC7.10 (GND), IC8.10 (GND), J1.3 (Pin_3), J1.4 (Pin_4), J3.25 (Pin_25), J3.26 (Pin_26), J3.27 (Pin_27), J3.28 (Pin_28), J3.29 (Pin_29), J3.30 (Pin_30), J4.23 (Pin_23), J4.24 (Pin_24), RN1.1 (R1.1), RN1.2 (R2.1), RN1.3 (R3.1), RN1.4 (R4.1), RN2.1 (R1.1), RN2.2 (R2.1), RN2.3 (R3.1), RN2.4 (R4.1), U3.1 (GND)
- net HALT: now also IC3.8 (A7)
- net IPL0: now also IC2.7 (A6)
- net IPL1: now also IC2.8 (A7)
- net IPL2: now also IC2.9 (A8)
- net LDS: now also IC1.7 (A6)
- net RESET: now also IC3.7 (A6)
- net RW: now also IC1.6 (A5)
- net UDS: now also IC1.8 (A7)
- net VMA: now also IC3.6 (A5)
- net VPA: now also IC3.4 (A3)
- new net +3V3: C1.1, C10.1, C2.1, C3.1, C4.1, C5.1, C6.1, C7.1, C8.1, IC1.20 (VCC), IC2.20 (VCC), IC3.20 (VCC), IC4.20 (VCC), IC5.20 (VCC), IC6.20 (VCC), IC7.20 (VCC), IC8.20 (VCC), J1.1 (Pin_1), J1.2 (Pin_2), U3.2 (VO)
- new net OE_A_L: IC4.19 (~{OE}), J3.35 (Pin_35), RN1.7 (R2.2)
- new net OE_A_M: IC5.19 (~{OE}), J3.37 (Pin_37), RN2.5 (R4.2)
- new net OE_A_U: IC6.19 (~{OE}), J3.39 (Pin_39), RN2.8 (R1.2)
- new net OE_C_1: IC1.19 (~{OE}), J3.32 (Pin_32), RN1.5 (R4.2)
- new net OE_C_2: IC2.19 (~{OE}), J3.34 (Pin_34), RN1.6 (R3.2)
- new net OE_C_3: IC3.19 (~{OE}), J3.36 (Pin_36), RN1.8 (R1.2)
- new net OE_D_L: IC7.19 (~{OE}), J3.38 (Pin_38), RN2.6 (R3.2)
- new net OE_D_U: IC8.19 (~{OE}), J3.40 (Pin_40), RN2.7 (R2.2)
- new net _A1: IC4.11 (B8), J3.1 (Pin_1)
- new net _A10: IC5.13 (B6), J3.10 (Pin_10)
- new net _A11: IC5.14 (B5), J3.11 (Pin_11)
- new net _A12: IC5.15 (B4), J3.12 (Pin_12)
- new net _A13: IC5.16 (B3), J3.13 (Pin_13)
- new net _A14: IC5.17 (B2), J3.14 (Pin_14)
- new net _A15: IC5.18 (B1), J3.15 (Pin_15)
- new net _A16: IC6.11 (B8), J3.16 (Pin_16)
- new net _A17: IC6.12 (B7), J3.17 (Pin_17)
- new net _A18: IC6.13 (B6), J3.18 (Pin_18)
- new net _A19: IC6.14 (B5), J3.19 (Pin_19)
- new net _A2: IC4.12 (B7), J3.2 (Pin_2)
- new net _A20: IC6.15 (B4), J3.20 (Pin_20)
- new net _A21: IC6.16 (B3), J3.21 (Pin_21)
- new net _A22: IC6.17 (B2), J3.22 (Pin_22)
- new net _A23: IC6.18 (B1), J3.23 (Pin_23)
- new net _A3: IC4.13 (B6), J3.3 (Pin_3)
- new net _A4: IC4.14 (B5), J3.4 (Pin_4)
- new net _A5: IC4.15 (B4), J3.5 (Pin_5)
- new net _A6: IC4.16 (B3), J3.6 (Pin_6)
- new net _A7: IC4.17 (B2), J3.7 (Pin_7)
- new net _A8: IC5.11 (B8), J3.8 (Pin_8)
- new net _A9: IC5.12 (B7), J3.9 (Pin_9)
- new net _AS: IC1.11 (B8), J4.18 (Pin_18)
- new net _BERR: IC3.17 (B2), J4.7 (Pin_7)
- new net _BG: IC1.16 (B3), J4.15 (Pin_15)
- new net _BGACK: IC1.17 (B2), J4.14 (Pin_14)
- new net _BR: IC1.18 (B1), J4.13 (Pin_13)
- new net _CLK: IC3.11 (B8), J4.22 (Pin_22)
- new net _D0: IC7.18 (B1), J4.25 (Pin_25)
- new net _D1: IC7.17 (B2), J4.26 (Pin_26)
- new net _D10: IC8.13 (B6), J4.35 (Pin_35)
- new net _D11: IC8.14 (B5), J4.36 (Pin_36)
- new net _D12: IC8.15 (B4), J4.37 (Pin_37)
- new net _D13: IC8.16 (B3), J4.38 (Pin_38)
- new net _D14: IC8.17 (B2), J4.39 (Pin_39)
- new net _D15: IC8.18 (B1), J4.40 (Pin_40)
- new net _D2: IC7.16 (B3), J4.27 (Pin_27)
- new net _D3: IC7.15 (B4), J4.28 (Pin_28)
- new net _D4: IC7.14 (B5), J4.29 (Pin_29)
- new net _D5: IC7.13 (B6), J4.30 (Pin_30)
- new net _D6: IC7.12 (B7), J4.31 (Pin_31)
- new net _D7: IC7.11 (B8), J4.32 (Pin_32)
- new net _D8: IC8.11 (B8), J4.33 (Pin_33)
- new net _D9: IC8.12 (B7), J4.34 (Pin_34)
- new net _DTACK: IC1.15 (B4), J4.16 (Pin_16)
- new net _E: IC3.15 (B4), J4.9 (Pin_9)
- new net _FC0: IC2.16 (B3), J4.1 (Pin_1)
- new net _FC1: IC2.15 (B4), J4.3 (Pin_3)
- new net _FC2: IC2.14 (B5), J4.5 (Pin_5)
- new net _HALT: IC3.12 (B7), J4.12 (Pin_12)
- new net _IPL0: IC2.13 (B6), J4.2 (Pin_2)
- new net _IPL1: IC2.12 (B7), J4.4 (Pin_4)
- new net _IPL2: IC2.11 (B8), J4.6 (Pin_6)
- new net _LDS: IC1.13 (B6), J4.19 (Pin_19)
- new net _RESET: IC3.13 (B6), J4.11 (Pin_11)
- new net _RW: IC1.14 (B5), J4.17 (Pin_17)
- new net _UDS: IC1.12 (B7), J4.20 (Pin_20)
- new net _VMA: IC3.14 (B5), J4.10 (Pin_10)
- new net _VPA: IC3.16 (B3), J4.8 (Pin_8)
- no-connect marks 4 -> 12
Other:
- title: 68K debug header breakout -> 68K 3V3 breakout
- moved on the sheet: J2

Commit message: Minor tweaks pre-gerberisation
Parts:
- J1, J2: footprint Connector_PinSocket_2.54mm:PinSocket_2x02_P2.54mm_Vertical -> Connector_PinHeader_2.54mm:PinHeader_2x02_P2.54mm_Vertical
Changed lines of the file:
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@@
     (property "Reference" "J2" (id 0) (at 318.77 224.9932 0))
     (property "Value" "Conn_02x02_Odd_Even" (id 1) (at 318.77 227.3046 0))
-    (property "Footprint" "Connector_PinSocket_2.54mm:PinSocket_2x02_P2.54mm_Vertical" (id 2) (at 317.5 230.505 0)
+    (property "Footprint" "Connector_PinHeader_2.54mm:PinHeader_2x02_P2.54mm_Vertical" (id 2) (at 317.5 230.505 0)
       (effects (font (size 1.27 1.27)) hide)
     )
@@
     (property "Reference" "J1" (id 0) (at 341.63 224.9932 0))
     (property "Value" "Conn_02x02_Odd_Even" (id 1) (at 341.63 227.3046 0))
-    (property "Footprint" "Connector_PinSocket_2.54mm:PinSocket_2x02_P2.54mm_Vertical" (id 2) (at 340.36 230.505 0)
+    (property "Footprint" "Connector_PinHeader_2.54mm:PinHeader_2x02_P2.54mm_Vertical" (id 2) (at 340.36 230.505 0)
       (effects (font (size 1.27 1.27)) hide)
     )
@@
     )
     (path "/57070c29-5005-4fdc-8062-b165957e0bf6"
-      (reference "J1") (unit 1) (value "Conn_02x02_Odd_Even") (footprint "Connector_PinSocket_2.54mm:PinSocket_2x02_P2.54mm_Vertical")
+      (reference "J1") (unit 1) (value "Conn_02x02_Odd_Even") (footprint "Connector_PinHeader_2.54mm:PinHeader_2x02_P2.54mm_Vertical")
     )
     (path "/00000000-0000-0000-0000-000062c3d0cb"
-      (reference "J2") (unit 1) (value "Conn_02x02_Odd_Even") (footprint "Connector_PinSocket_2.54mm:PinSocket_2x02_P2.54mm_Vertical")
+      (reference "J2") (unit 1) (value "Conn_02x02_Odd_Even") (footprint "Connector_PinHeader_2.54mm:PinHeader_2x02_P2.54mm_Vertical")
     )
     (path "/68661299-5104-4868-aadf-f82ed2983f63"
