File: 68k_cpld_devboard.kicad_pcb (KiCad board)
At the start: 2 copper layers, 17 parts, among them J1 Conn_01x10_Socket, J2 Conn_01x10_Socket, J3 Conn_01x06_Pin, U1 68000D_PLUG, U2 68000D, U3 LM1117MP-3.3, U4 XC95144XL-TQ100

Commit message: Passing DRC
Parts:
- added TP1: TestPoint_Small, TestPoint:TestPoint_Pad_D1.0mm, B.Cu at (63.5, 39.4)
- J1: value Conn_01x10_Socket -> Conn_02x10_Odd_Even; footprint Connector_PinSocket_2.54mm:PinSocket_2x05_P2.54mm_Vertical -> Connector_PinSocket_2.54mm:PinSocket_2x10_P2.54mm_Vertical
- J2: value Conn_01x10_Socket -> Conn_01x03_Pin; footprint Connector_PinSocket_2.54mm:PinSocket_2x05_P2.54mm_Vertical -> Connector_PinHeader_2.54mm:PinHeader_1x03_P2.54mm_Vertical
- J3: footprint Connector_PinHeader_2.54mm:PinHeader_1x06_P2.54mm_Horizontal -> Connector_PinHeader_2.54mm:PinHeader_1x06_P2.54mm_Vertical
- moved J1 62.6 mm to (29.1, 34.0), turned to 90 degrees
- moved J2 29.8 mm to (29.2, 52.8), turned to 180 degrees
- moved C8 8.64 mm to (38.4, 52.8), turned to 0 degrees
- moved C9 6.80 mm to (38.4, 50.4), turned to 0 degrees
- moved U3 6.70 mm to (38.1, 50.3), turned to 0 degrees
Connections:
- J1 pad 1: Net-(J1-Pin_1) -> /P73
- J1 pad 10: Net-(J1-Pin_10) -> /P55
- J1 pad 2: Net-(J1-Pin_2) -> /P50
- J1 pad 3: Net-(J1-Pin_3) -> /P72
- J1 pad 4: Net-(J1-Pin_4) -> /P52
- J1 pad 5: Net-(J1-Pin_5) -> /P71
- J1 pad 6: Net-(J1-Pin_6) -> /P53
- J1 pad 7: Net-(J1-Pin_7) -> /P70
- J1 pad 8: Net-(J1-Pin_8) -> /P54
- J1 pad 9: Net-(J1-Pin_9) -> /P68
- J2 pad 1: Net-(J2-Pin_1) -> +5V
- J2 pad 2: Net-(J2-Pin_2) -> +3V3
- J2 pad 3: Net-(J2-Pin_3) -> GND
- U4 pad 50: Net-(J1-Pin_1) -> /P50
- U4 pad 52: Net-(J1-Pin_2) -> /P52
- U4 pad 53: Net-(J1-Pin_3) -> /P53
- U4 pad 54: Net-(J1-Pin_4) -> /P54
- U4 pad 55: Net-(J1-Pin_5) -> /P55
- U4 pad 56: Net-(J1-Pin_6) -> /P56
- U4 pad 58: Net-(J1-Pin_7) -> /P58
- U4 pad 59: Net-(J1-Pin_8) -> /P59
- U4 pad 60: Net-(J1-Pin_9) -> /P60
- U4 pad 61: Net-(J1-Pin_10) -> /P61
- U4 pad 63: Net-(J2-Pin_1) -> /P63
- U4 pad 64: Net-(J2-Pin_2) -> /P64
- U4 pad 65: Net-(J2-Pin_3) -> /P65
- U4 pad 66: Net-(J2-Pin_4) -> /P66
- U4 pad 67: Net-(J2-Pin_5) -> /P67
- U4 pad 68: Net-(J2-Pin_6) -> /P68
- U4 pad 70: Net-(J2-Pin_7) -> /P70
- U4 pad 71: Net-(J2-Pin_8) -> /P71
- U4 pad 72: Net-(J2-Pin_9) -> /P72
- U4 pad 73: Net-(J2-Pin_10) -> /P73
- U4 pad 74: unconnected-(U4-P74-Pad74) -> /P74
Routing:
- net /P50: track 0.00 -> 54.1 mm, vias 0 -> 1
- net /P52: track 0.00 -> 53.3 mm, vias 0 -> 1
- net /P53: track 0.00 -> 49.0 mm, vias 0 -> 1
- net /TDO: track 0.00 -> 46.4 mm, vias 0 -> 2
- net +3V3: track 77.6 -> 122.6 mm
- net /P54: track 0.00 -> 44.9 mm, vias 0 -> 1
- net /P73: track 0.00 -> 41.2 mm
- net /P55: track 0.00 -> 40.8 mm, vias 0 -> 1
- net /P72: track 0.00 -> 39.1 mm
- net /P71: track 0.00 -> 37.3 mm
- net /P56: track 0.00 -> 36.7 mm, vias 0 -> 1
- net /TMS: track 0.00 -> 35.4 mm, vias 0 -> 1
- net /P70: track 0.00 -> 35.2 mm
- net /P68: track 0.00 -> 33.6 mm
- net /P58: track 0.00 -> 32.8 mm, vias 0 -> 1
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- added copper zone on B.Cu, net GND
Other:
- board outline added: 82.3 x 56.4 mm
- board text added: "3V3 GND TCK TDO TDI TMS"
- board text added: "Copyright 2024 D Henderson github.com/dh219"
- board text added: "GND 3V3 5V"
- board text added: "P50 P52 P53 P54 P55 P56 P58 P59 P60 P61"
- board text added: "P73 P72 P71 P70 P68 P67 P66 P65 P64 P63"
- board text added: "~{68k CPLD DEVBOARD}"
- board text removed: "Copyright 2023 D Henderson github.com/dh219"
- board text removed: "~{68k BREAKOUT 3V3}"
