File: 68k_cpld_devboard.kicad_sch (KiCad schematic)
At the start: 17 parts, among them J1 Conn_01x10_Socket, J2 Conn_01x10_Socket, J3 Conn_01x06_Pin, U1 68000D_PLUG, U2 68000D, U3 LM1117MP-3.3, U4 XC95144XL-TQ100

Commit message: Passing DRC
Parts:
- removed J1, J2: Conn_01x10_Socket, Connector_PinSocket_2.54mm:PinSocket_2x05_P2.54mm_Vertical, symbol Connector:Conn_01x10_Socket
- added J1: Conn_02x10_Odd_Even, Connector_PinSocket_2.54mm:PinSocket_2x10_P2.54mm_Vertical, symbol Connector_Generic:Conn_02x10_Odd_Even
- added J2: Conn_01x03_Pin, Connector_PinHeader_2.54mm:PinHeader_1x03_P2.54mm_Vertical, symbol Connector:Conn_01x03_Pin
- added TP1: TestPoint_Small, TestPoint:TestPoint_Pad_D1.0mm, symbol Connector:TestPoint_Small
- J3: footprint Connector_PinHeader_2.54mm:PinHeader_1x06_P2.54mm_Horizontal -> Connector_PinHeader_2.54mm:PinHeader_1x06_P2.54mm_Vertical
Connections:
- net +3V3: now also J2.2 (Pin_2)
- net +5V: now also J2.1 (Pin_1)
- net GND: now also J2.3 (Pin_3)
- net P63: now reaches U4.63 (P63)
- net P63: now also J1.19 (Pin_19)
- net P73: now reaches U4.73 (P73)
- net P73: now also J1.1 (Pin_1)
- net P64: now reaches U4.64 (P64)
- net P64: now also J1.17 (Pin_17)
- net P65: now reaches U4.65 (P65)
- net P65: now also J1.15 (Pin_15)
- net P66: now reaches U4.66 (P66)
- net P66: now also J1.13 (Pin_13)
- net P67: now reaches U4.67 (P67)
- net P67: now also J1.11 (Pin_11)
- net P68: now reaches U4.68 (P68)
- net P68: now also J1.9 (Pin_9)
- net P70: now reaches U4.70 (P70)
- net P70: now also J1.7 (Pin_7)
- net P71: now reaches U4.71 (P71)
- net P71: now also J1.5 (Pin_5)
- net P72: now reaches U4.72 (P72)
- net P72: now also J1.3 (Pin_3)
- net P50: now reaches U4.50 (P50)
- net P50: now also J1.2 (Pin_2)
- net P52: now reaches U4.52 (P52)
- net P52: now also J1.4 (Pin_4)
- net P53: now reaches U4.53 (P53)
- net P53: now also J1.6 (Pin_6)
- net P54: now reaches U4.54 (P54)
- net P54: now also J1.8 (Pin_8)
- net P55: now reaches U4.55 (P55)
- net P55: now also J1.10 (Pin_10)
- net P56: now reaches U4.56 (P56)
- net P56: now also J1.12 (Pin_12)
- net P58: now reaches U4.58 (P58)
- net P58: now also J1.14 (Pin_14)
- net P59: now reaches U4.59 (P59)
- net P59: now also J1.16 (Pin_16)
- net P60: now reaches U4.60 (P60)
- net P60: now also J1.18 (Pin_18)
- net P61: now reaches U4.61 (P61)
- net P61: now also J1.20 (Pin_20)
- net P74: now reaches U4.74 (P74)
- net P74: now also TP1.1
